Commit message: add lidar and imu sensor

File: hunter_se/hunter_se_description/urdf/hunter_hw_interface.xacro (robot description, xacro)
@@ -7,7 +7,9 @@
             <xacro:if value="${tf_prefix == ''}">
                 <xacro:property name="joint_prefix" value=""/>
+                <xacro:property name="file_prefix" value="base"/>
             </xacro:if>
             <xacro:unless value="${tf_prefix == ''}">
                 <xacro:property name="joint_prefix" value="${tf_prefix}/"/>
+                <xacro:property name="file_prefix" value="${tf_prefix}"/>
             </xacro:unless>
             <xacro:if value="${simulation}">
@@ -68,5 +70,5 @@
                     <namespace>${tf_prefix}</namespace>
                 </ros>
-                <parameters>$(find hunter_se_description)/config/${tf_prefix}_controllers.yaml</parameters>
+                <parameters>$(find hunter_se_description)/config/${file_prefix}_controllers.yaml</parameters>
             </plugin>
         </gazebo>

File: hunter_se/hunter_se_description/urdf/hunter_se_alone.xacro (robot description, xacro)
@@ -3,7 +3,11 @@
     <xacro:include filename="$(find hunter_se_description)/urdf/hunter_se_macro.xacro"/>
     <xacro:include filename="$(find hunter_se_description)/urdf/hunter_hw_interface.xacro"/>
+    <xacro:include filename="$(find hunter_se_description)/urdf/lidar_sensor.xacro"/>
+    <xacro:include filename="$(find hunter_se_description)/urdf/imu_sensor.xacro"/>
     <xacro:arg name="tf_prefix" default=""/>
     <xacro:arg name="simulation" default="true"/>
     <xacro:hunter_se tf_prefix="$(arg tf_prefix)" simulation="$(arg simulation)"/>
     <xacro:hunter_se_hw_int tf_prefix="$(arg tf_prefix)" simulation="$(arg simulation)"/>
+    <xacro:lidar_sensor tf_prefix="$(arg tf_prefix)"/>
+    <xacro:imu_sensor tf_prefix="$(arg tf_prefix)"/>
 </robot>

File: hunter_se/hunter_se_description/urdf/hunter_se_macro.xacro (robot description, xacro)
@@ -162,9 +162,9 @@
                     rpy="0 0 0" />
                 <geometry>
-                    <cylinder length="0.001" radius="0.135" />
+                    <cylinder length="0.01" radius="0.135" />
                     <!-- <mesh
                     filename="package://hunter_se_description/meshes/fr_left_link_coll.STL" /> -->
                 </geometry>
-                <xacro:wheels_collision mu="1.0" slip="1.0"/>
+                <xacro:wheels_collision mu="100.0" slip="1.0"/>
             </collision>
         </link>
@@ -254,9 +254,9 @@
                     rpy="0 0 0" />
                 <geometry>
-                    <cylinder length="0.001" radius="0.135" />
+                    <cylinder length="0.01" radius="0.135" />
                     <!-- <mesh
                     filename="package://hunter_se_description/meshes/fr_right_link_coll.STL" /> -->
                 </geometry>
-                 <xacro:wheels_collision mu="1.0" slip="1.0"/>
+                 <xacro:wheels_collision mu="100.0" slip="1.0"/>
             </collision>
         </link>
@@ -307,9 +307,9 @@
                     rpy="0 0 0" />
                 <geometry>
-                    <cylinder length="0.001" radius="0.135" />
+                    <cylinder length="0.01" radius="0.135" />
                     <!-- <mesh
                     filename="package://hunter_se_description/meshes/re_left_link_coll.STL" /> -->
                 </geometry>
-                <xacro:wheels_collision mu="1.0" slip="1.0"/>
+                <xacro:wheels_collision mu="100.0" slip="1.0"/>
             </collision>
         </link>
@@ -362,9 +362,9 @@
                     rpy="0 0 0" />
                 <geometry>
-                    <cylinder length="0.001" radius="0.135" />
+                    <cylinder length="0.01" radius="0.135" />
                     <!-- <mesh
                     filename="package://hunter_se_description/meshes/re_right_link_coll.STL" /> -->
                 </geometry>
-                 <xacro:wheels_collision mu="1.0" slip="1.0"/>
+                 <xacro:wheels_collision mu="100.0" slip="1.0"/>
             </collision>
         </link>
